File: PandaputeKiCad/Pandapute.kicad_pcb (KiCad board)
At the start: 4 copper layers, 191 x 158 mm, 131 parts, among them IC1 ES8311, J1 Conn_01x02_Pin, J10 Conn_01x04_Pin, J2 USB_C_Receptacle_USB2.0_16P, J3 Conn_01x02_Pin, J4 PJ-342B, J5 Conn_01x14_Pin, J6 Conn_01x04_Pin, J7 Conn_01x03_Pin, J8 Conn_01x05_Pin, J9 Conn_01x04_Pin, SW1 SW_Push, SW10 SW_Push, SW11 SW_Push, SW12 SW_Push, SW13 SW_Push, SW14 SW_Push, SW15 SW_Push, SW16 SW_Push, SW17 SW_Push, SW18 SW_Push, SW19 SW_Push, SW2 SW_Push, SW20 SW_Push, SW21 SW_Push, SW22 SW_Push, SW23 SW_Push, SW24 SW_Push, SW25 SW_Push, SW26 SW_Push, SW27 SW_Push, SW28 SW_Push, SW29 SW_Push, SW3 SW_Push, SW30 SW_Push, SW31 SW_Push, SW32 SW_Push, SW33 SKRHABE010, SW4 SW_Push, SW5 SW_Push, SW6 SW_Push, SW7 SW_Push, SW8 SW_Push, SW9 SW_Push, U1 AP2112K-3.3, U2 IP5306, U3 ESP32-S3-WROOM-1, U4 NS4150, U5 TCA8418RTWR, U6 MPU-6050

Commit message: adding PCB 3D model screenshots for visualization
Parts:
- J6: footprint Connector_PinSocket_2.54mm:PinSocket_1x04_P2.54mm_Vertical -> Connector_PinHeader_2.54mm:PinHeader_1x04_P2.54mm_Vertical
